Commit message: added frame task gain, solver daming value to ik removed posture task cleaned styling for precommit

File: piper_description/urdf/piper_description.urdf (robot description, URDF)
Before this commit: robot piper, 12 links, 11 joints
Joints:
- joint joint1: limit lower=-2.618 upper=2.618 effort=100 velocity=15 -> lower=-2.618 upper=2.618 effort=100 velocity=10
- joint joint2: limit lower=0 upper=3.14 effort=100 velocity=15 -> lower=0 upper=3.14 effort=100 velocity=10
- joint joint3: limit lower=-2.967 upper=0 effort=100 velocity=15 -> lower=-2.967 upper=0 effort=100 velocity=10
- joint joint4: limit lower=-1.745 upper=1.745 effort=100 velocity=15 -> lower=-1.745 upper=1.745 effort=100 velocity=10
- joint joint5: limit lower=-1.22 upper=1.22 effort=100 velocity=15 -> lower=-1.22 upper=1.22 effort=100 velocity=10
- joint joint6: limit lower=-2.0944 upper=2.0944 effort=100 velocity=15 -> lower=-2.0944 upper=2.0944 effort=100 velocity=10
